File: hardware/temperature-ir-v2.kicad_pcb (KiCad board)
At the start: 2 copper layers, 20 x 25 mm, 24 parts, among them P1 CON-SENSOR2, P2 DEBUG, P3 BOOT, U1 XMC110024, U2 MLX90614, U4 DRILL, U5 DRILL, U6 DRILL, U7 DRILL

Commit message: fix status text
Other:
- board text added: "Status"
- board text removed: "status"
Changed lines of the file:
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@@
   )
   (layers
-    (0 Vorderseite signal)
-    (31 Rückseite signal)
+    (0 Vorderseite signal hide)
+    (31 Rückseite signal hide)
     (32 B.Adhes user)
     (33 F.Adhes user)
@@
   )
   (gr_circle (center 118.88 107.26) (end 123.08 107.26) (layer Dwgs.User) (width 0.381))
-  (gr_text status (at 124.18 112.26) (layer F.SilkS)
+  (gr_text Status (at 124.18 112.26) (layer F.SilkS)
     (effects (font (size 0.8001 0.8001) (thickness 0.14986)))
   )
