File: hardware/temperature-ir-v2.kicad_pcb (KiCad board)
At the start: 2 copper layers, 20 x 25 mm, 24 parts, among them P1 CON-SENSOR2, P2 DEBUG, P3 BOOT, U1 XMC110024, U2 MLX90614, U4 DRILL, U5 DRILL, U6 DRILL, U7 DRILL

Commit message: move to new kicad version
Other:
- net class Default removed
